File: STMCastomBoard.kicad_sch (KiCad schematic)
At the start: 2 parts, among them U1 W9825G6KH-6, U2 STM32H743IITx

Commit message: adding main parts
Parts:
- added C1, C2: 4.7uF, Capacitor_SMD:C_0201_0603Metric_Pad0.64x0.40mm_HandSolder, symbol Device:C_Small
- added C10, C3, C4, C5, C6, C7, C8, C9: 0.1uF, Capacitor_SMD:C_0201_0603Metric_Pad0.64x0.40mm_HandSolder, symbol Device:C_Small
- added F1: Fuse_Small, Fuse:Fuse_0603_1608Metric_Pad1.05x0.95mm_HandSolder, symbol Device:Fuse_Small
- added FL1, FL2: BLM21PG220SN1D, BLM21PG220SN1D:BEADC2012X105N, symbol BLM21PG220SN1D:BLM21PG220SN1D
- added J1: FH55M-40S-0.4SH, FH55M-40S-0.4SH:HRS_FH55M-40S-0.4SH, symbol FH55M-40S-0.4SH:FH55M-40S-0.4SH
- added R1, R2: 10K, Resistor_SMD:R_0201_0603Metric_Pad0.64x0.40mm_HandSolder, symbol Device:R
- added U3: AP7361C-33E, Package_TO_SOT_SMD:SOT-223-3_TabPin2, symbol Regulator_Linear:AP7361C-33E
- added U4: W25Q128JVS, Package_SO:SOIC-8_5.3x5.3mm_P1.27mm, symbol Memory_Flash:W25Q128JVS
- added U5: CH340X, Package_SO:MSOP-10_3x3mm_P0.5mm, symbol Interface_USB:CH340X
Connections:
- net SDRAM33: now reaches U1.1 (VDD), U1.14 (VDD), U1.27 (VDD)
- net SDRAM33: now also U1.3 (VDDQ), U1.43 (VDDQ), U1.49 (VDDQ), U1.9 (VDDQ), C3.1, C4.1, C5.1, C6.1, C7.1, C8.1, C9.1, FL1.1, R1.2
- net DQ5: now reaches U1.10 (DQ5)
- net DQ5: now also U2.69 (PE8)
- net DQ6: now reaches U1.11 (DQ6)
- net DQ6: now also U2.70 (PE9)
- net GND: now reaches U1.12 (VSSQ), U1.46 (VSSQ), U1.52 (VSSQ), U1.6 (VSSQ)
- net GND: now also U1.28 (VSS), U1.41 (VSS), U1.54 (VSS), C1.2, C10.1, C2.2, C3.2, C4.2, C5.2, C6.2, C7.2, C8.2, C9.2, J1.29, J1.3, J1.36, U3.2 (GND), U4.4 (GND)
- net DQ7: now reaches U1.13 (DQ7)
- net DQ7: now also U2.73 (PE10)
- net NBL0: now reaches U1.15 (LDQM)
- net NBL0: now also U2.169 (PE0)
- net SDNWE: now reaches U1.16 (~{WE})
- net SDNWE: now also U2.32 (PC0)
- net SDNCAS: now reaches U1.17 (~{CAS})
- net SDNCAS: now also U2.160 (PG15)
- net SDNRAS: now reaches U1.18 (~{RAS})
- net SDNRAS: now also U2.59 (PF11)
- net SDNCS: now reaches U1.19 (~{CS})
- net SDNCS: now also U2.44 (PH3), R1.1
- net DQ0: now reaches U1.2 (DQ0)
- net DQ0: now also U2.104 (PD14)
- net BS0: now reaches U1.20 (BS0)
- net BS0: now also U2.108 (PG4)
- net BS1: now reaches U1.21 (BS1)
- net BS1: now also U2.109 (PG5)
- net A10: now reaches U1.22 (A10/AP)
- net A10: now also U2.66 (PG0)
- net A0: now reaches U1.23 (A0)
- net A0: now also U2.16 (PF0)
- net A1: now reaches U1.24 (A1)
- net A1: now also U2.17 (PF1)
- net A2: now reaches U1.25 (A2)
- net A2: now also U2.18 (PF2)
- net A3: now reaches U1.26 (A3)
- net A3: now also U2.19 (PF3)
- net A4: now reaches U1.29 (A4)
- net A4: now also U2.20 (PF4)
- net A5: now reaches U1.30 (A5)
- net A5: now also U2.21 (PF5)
- net A6: now reaches U1.31 (A6)
- net A6: now also U2.60 (PF12)
- net A7: now reaches U1.32 (A7)
- net A7: now also U2.63 (PF13)
- net A8: now reaches U1.33 (A8)
- net A8: now also U2.64 (PF14)
- net A9: now reaches U1.34 (A9)
- net A9: now also U2.65 (PF15)
- net A11: now reaches U1.35 (A11)
- net A11: now also U2.67 (PG1)
- net A12: now reaches U1.36 (A12)
- net A12: now also U2.106 (PG2)
- net SDNCKE: now reaches U1.37 (CKE)
- net SDNCKE: now also U2.43 (PH2)
- net SDNCLK: now reaches U1.38 (CLK)
- net SDNCLK: now also U2.112 (PG8)
- net NBL1: now reaches U1.39 (UDQM)
- net NBL1: now also U2.170 (PE1)
- net DQ1: now reaches U1.4 (DQ1)
- net DQ1: now also U2.105 (PD15)
- net DQ8: now reaches U1.42 (DQ8)
- net DQ8: now also U2.74 (PE11)
- net DQ9: now reaches U1.44 (DQ9)
- net DQ9: now also U2.75 (PE12)
- net DQ10: now reaches U1.45 (DQ10)
- net DQ10: now also U2.76 (PE13)
- net DQ11: now reaches U1.47 (DQ11)
- net DQ11: now also U2.77 (PE14)
- net DQ12: now reaches U1.48 (DQ12)
- net DQ12: now also U2.78 (PE15)
- net DQ2: now reaches U1.5 (DQ2)
- net DQ2: now also U2.142 (PD0)
- net DQ13: now reaches U1.50 (DQ13)
- net DQ13: now also U2.96 (PD8)
- net DQ14: now reaches U1.51 (DQ14)
- net DQ14: now also U2.97 (PD9)
- net DQ15: now reaches U1.53 (DQ15)
- net DQ15: now also U2.98 (PD10)
- net DQ3: now reaches U1.7 (DQ3)
- net DQ3: now also U2.143 (PD1)
- net DQ4: now reaches U1.8 (DQ4)
- net DQ4: now also U2.68 (PE7)
- net TP_SDA: now reaches U2.100 (PD12)
- net TP_SDA: now also J1.37
- net TP_SCL: now reaches U2.101 (PD13)
- net TP_SCL: now also J1.38
- net LCD_VSYNC: now reaches U2.11 (PI9)
- net LCD_VSYNC: now also J1.33
- net LCD_R7: now reaches U2.110 (PG6)
- net LCD_R7: now also J1.12
- net LCD_DCLK: now reaches U2.111 (PG7)
- net LCD_DCLK: now also J1.30
- net LCD_B3: now reaches U2.119 (PA8)
- net LCD_B3: now also J1.24
- net LCD_HSYNC: now reaches U2.12 (PI10)
- net LCD_HSYNC: now also J1.32
- net LCD_G2: now reaches U2.128 (PH13)
- net LCD_G2: now also J1.15
- net LCD_G3: now reaches U2.129 (PH14)
- net LCD_G3: now also J1.16
- net LCD_G4: now reaches U2.130 (PH15)
- net LCD_G4: now also J1.17
- net LCD_G5: now reaches U2.131 (PI0)
- net LCD_G5: now also J1.18
- net LCD_G6: now reaches U2.132 (PI1)
- net LCD_G6: now also J1.19
- net LCD_G7: now reaches U2.133 (PI2)
- net LCD_G7: now also J1.20
- net LCD_B2: now reaches U2.150 (PD6)
- net LCD_B2: now also J1.23
- net TP_INT: now reaches U2.151 (PD7)
- net TP_INT: now also J1.40
- net LCD_B1: now reaches U2.155 (PG12)
- net LCD_B1: now also J1.22
- net LCD_R0: now reaches U2.156 (PG13)
- net LCD_R0: now also J1.5
- net LCD_B0: now reaches U2.157 (PG14)
- net LCD_B0: now also J1.21
- net LCD_PWM (GPIO Output): now reaches U2.163 (PB5)
- net LCD_PWM (GPIO Output): now also J1.35
- net QSPI_BK1_CS: now reaches U2.164 (PB6)
- net QSPI_BK1_CS: now also R2.2, U4.1 (~{CS})
- net LCD_B4: now reaches U2.173 (PI4)
- net LCD_B4: now also J1.25
- net LCD_B5: now reaches U2.174 (PI5)
- net LCD_B5: now also J1.26
- net LCD_B6: now reaches U2.175 (PI6)
- net LCD_B6: now also J1.27
- net LCD_B7: now reaches U2.176 (PI7)
- net LCD_B7: now also J1.28
- net QSPI_BK1_IO3: now reaches U2.24 (PF6)
- net QSPI_BK1_IO3: now also U4.7 (~{HOLD}/~{RESET}/IO_{3})
- net QSPI_BK1_IO2: now reaches U2.25 (PF7)
- net QSPI_BK1_IO2: now also U4.3 (~{WP}/IO_{2})
- net QSPI_BK1_IO0: now reaches U2.26 (PF8)
- net QSPI_BK1_IO0: now also U4.5 (DI/IO_{0})
- net QSPI_BK1_IO1: now reaches U2.27 (PF9)
- net QSPI_BK1_IO1: now also U4.2 (DO/IO_{1})
- net LCD_DE: now reaches U2.28 (PF10)
- net LCD_DE: now also J1.34
- net LCD_G0: now reaches U2.4 (PE5)
- net LCD_G0: now also J1.13
- net LCD_R1: now reaches U2.42 (PA2)
- net LCD_R1: now also J1.6
- net LCD_G1: now reaches U2.5 (PE6)
- net LCD_G1: now also J1.14
- net QSPI_BK1_CLK: now reaches U2.58 (PB2)
- net QSPI_BK1_CLK: now also U4.6 (CLK)
- net LCD_R2: now reaches U2.85 (PH8)
- net LCD_R2: now also J1.7
- net LCD_R3: now reaches U2.86 (PH9)
- net LCD_R3: now also J1.8
- net LCD_R4: now reaches U2.87 (PH10)
- net LCD_R4: now also J1.9
- net LCD_R5: now reaches U2.88 (PH11)
- net LCD_R5: now also J1.10
- net LCD_R6: now reaches U2.89 (PH12)
- net LCD_R6: now also J1.11
- net TP_RST: now reaches U2.99 (PD11)
- net TP_RST: now also J1.39
- new net: FL2.1, J1.1, J1.2
- new net VBUS: F1.1
- new net VDD: C1.1, F1.2, FL2.2, U3.1 (VI)
- new net VDD33: C10.2, C2.1, FL1.2, J1.31, J1.4, R2.1, U3.3 (VO), U4.8 (VCC)
Other:
- note added: "For ERC only"
- note added: "LCD-RGB interface"
- note added: "Power"
- note added: "QSPI FLASH"
- note added: "SDRAM"
- moved on the sheet: U1, U2
